File: Hardware/1.81_Greyscale_OLED_Breakout.brd (EAGLE design)
At the start: 15.2 x 35.6 mm, 25 parts, among them U1 AP3012, U2 3.3V, U3 TXB0104

Commit message: Fixed issue with multiple boards
Parts:
- added FD3, FD4: FIDUCIAL1X2, SparkFun-Aesthetics:FIDUCIAL-1X2
- added LOGO2: REVISION, SparkFun-Aesthetics:REVISION
- added LOGO3: SFE_LOGO_FLAME.1_INCH, SparkFun-Aesthetics:SFE_LOGO_FLAME_.1
- C2: value 1.0uF/25V -> 1.0uF
- DS1: device 1.81_Greyscale_OLED_Breakout:OEL_1.8_FPC_Y3B -> SparkFun-Displays:OEL_1.8_FPC_Y3B
- LOGO1: value SPARKX-LOGO5 -> SFE_LOGO_NAME_FLAME.1_INCH; device 1.81_Greyscale_OLED_Breakout:SPARKX-LARGE -> SparkFun-Aesthetics:SFE_LOGO_NAME_FLAME_.1
- U1: value AP3012 -> 1.25V 500mA; device 1.81_Greyscale_OLED_Breakout:SOT23-5 -> SparkFun-IC-Power:SOT23-5
- moved FRAME1 26.7 mm to (-22.9, -8.89)
- moved LOGO1 6.11 mm to (13.6, 22.9)
- moved FD2 4.35 mm to (5.08, 34.3)
Other:
- board text added: "A. England"
- board text added: "v01"
Changed lines of the file:
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@@
 <text x="3.81" y="2.54" size="1.016" layer="21" ratio="15" rot="R90" align="center-left">SCLK</text>
 <text x="8.89" y="2.54" size="1.016" layer="21" ratio="15" rot="R90" align="center-left">!RES!</text>
-<text x="6.985" y="26.67" size="1.016" layer="22" ratio="15" rot="MR180" align="center">1.81" Greyscale
+<text x="7.112" y="29.718" size="1.016" layer="22" ratio="15" rot="MR180" align="center">1.81" Greyscale
 OLED Breakout</text>
-<text x="34.29" y="-10.16" size="1.778" layer="21" font="vector" ratio="15">N. Seidle</text>
+<text x="7.62" y="-8.89" size="1.778" layer="51" font="vector">N. Seidle</text>
+<text x="7.62" y="-11.43" size="1.778" layer="51" font="vector">A. England</text>
+<text x="1.651" y="8.509" size="1.27" layer="16" ratio="15" rot="MR270">v01</text>
 </plain>
 <attributes>
@@
 </autorouter>
 <elements>
-<element name="FRAME1" library="SparkFun-Aesthetics" package="CREATIVE_COMMONS" value="FRAME-LETTER" x="3.81" y="-10.16"/>
-<element name="U1" library="1.81_Greyscale_OLED_Breakout" package="SOT23-5" value="AP3012" x="11.43" y="29.21"/>
+<element name="FRAME1" library="SparkFun-Aesthetics" package="CREATIVE_COMMONS" value="FRAME-LETTER" x="-22.86" y="-8.89"/>
+<element name="U1" library="SparkFun-IC-Power" package="SOT23-5" value="1.25V 500mA" x="11.43" y="29.21">
+<attribute name="PROD_ID" value="VREG-13911" x="11.43" y="29.21" size="1.778" layer="27" display="off"/>
+<attribute name="VALUE" value="1.25V 500mA" x="11.43" y="29.21" size="1.778" layer="27" display="off"/>
+</element>
 <element name="C1" library="SparkFun-Capacitors" package="0603" value="1.0uF" x="11.43" y="32.639" rot="R180">
 <attribute name="PROD_ID" value="CAP-00868" x="11.43" y="32.639" size="1.778" layer="27" font="vector" ratio="15" rot="R180" display="off"/>
 </element>
-<element name="C2" library="SparkFun-Capacitors" package="0805" value="1.0uF/25V" x="11.43" y="22.86" smashed="yes" rot="R270">
-<attribute name="PROD_ID" value="CAP-11625" x="11.43" y="22.86" size="1.778" layer="27" font="vector" ratio="15" rot="R270" display="off"/>
+<element name="C2" library="SparkFun-Capacitors" package="0805" value="1.0uF" x="11.43" y="22.86" smashed="yes" rot="R270">
+<attribute name="PROD_ID" value="CAP-08064" x="11.43" y="22.86" size="1.778" layer="27" font="vector" ratio="15" rot="R270" display="off"/>
 <attribute name="NAME" x="12.319" y="22.86" size="0.6096" layer="25" font="vector" ratio="20" rot="R270" align="bottom-center"/>
 <attribute name="VALUE" x="14.478" y="22.86" size="0.6096" layer="27" font="vector" ratio="20" rot="R270" align="top-center"/>
@@
 </element>
 <element name="J2" library="SparkFun-Connectors" package="1X06_NO_SILK" value="" x="1.27" y="1.27" rot="MR180"/>
-<element name="LOGO1" library="1.81_Greyscale_OLED_Breakout" package="SPARKX-LARGE" value="SPARKX-LOGO5" x="7.493" y="23.241" rot="MR0"/>
+<element name="LOGO1" library="SparkFun-Aesthetics" package="SFE_LOGO_NAME_FLAME_.1" value="SFE_LOGO_NAME_FLAME.1_INCH" x="13.589" y="22.86" rot="MR0"/>
 <element name="H2" library="SparkFun-Hardware" package="STAND-OFF" value="STAND-OFF" x="2.54" y="33.02"/>
 <element name="FD1" library="SparkFun-Aesthetics" package="FIDUCIAL-1X2" value="FIDUCIAL1X2" x="12.7" y="5.715"/>
-<element name="FD2" library="SparkFun-Aesthetics" package="FIDUCIAL-1X2" value="FIDUCIAL1X2" x="0.762" y="34.798"/>
-<element name="DS1" library="1.81_Greyscale_OLED_Breakout" package="OEL_1.8_FPC_Y3B" value="OEL_1.8OEL_Y3B" x="7.62" y="31.75" rot="MR0"/>
+<element name="FD2" library="SparkFun-Aesthetics" package="FIDUCIAL-1X2" value="FIDUCIAL1X2" x="5.08" y="34.29"/>
+<element name="DS1" library="SparkFun-Displays" package="OEL_1.8_FPC_Y3B" value="OEL_1.8OEL_Y3B" x="7.62" y="31.75" rot="MR0">
+<attribute name="PROD_ID" value="LCD-13910" x="7.62" y="31.75" size="1.778" layer="28" rot="MR0" display="off"/>
+</element>
+<element name="LOGO2" library="SparkFun-Aesthetics" package="REVISION" value="REVISION" x="-11.43" y="-11.43"/>
+<element name="FD3" library="SparkFun-Aesthetics" package="FIDUCIAL-1X2" value="FIDUCIAL1X2" x="12.7" y="5.715" rot="MR0"/>
+<element name="FD4" library="SparkFun-Aesthetics" package="FIDUCIAL-1X2" value="FIDUCIAL1X2" x="5.08" y="34.29" rot="MR0"/>
+<element name="LOGO3" library="SparkFun-Aesthetics" package="SFE_LOGO_FLAME_.1" value="SFE_LOGO_FLAME.1_INCH" x="6.477" y="31.369"/>
 </elements>
 <signals>
