File: Hardware/1.81_Greyscale_OLED_Breakout.sch (EAGLE design)
At the start: 25 parts, among them U1 AP3012, U2 3.3V, U3 TXB0104

Commit message: Fixed issue with multiple boards
Parts:
- added FD3, FD4: FIDUCIAL1X2, SparkFun-Aesthetics:FIDUCIAL1X2
- added LOGO2: REVISION, SparkFun-Aesthetics:REVISION
- added LOGO3: SFE_LOGO_FLAME.1_INCH, SparkFun-Aesthetics:SFE_LOGO_FLAME.1_INCH
- C2: value 1.0uF/25V -> 1.0uF; device SparkFun-Capacitors:1.0UF-0805-25V-(+80/-20%) -> SparkFun-Capacitors:1.0UF-0805-25V-10%
- DS1: device 1.81_Greyscale_OLED_Breakout:OEL_1.8OEL_Y3B -> SparkFun-Displays:OEL_1.8OEL_Y3B
- L1: device 1.81_Greyscale_OLED_Breakout:INDUCTORINDUCTOR_10UH -> SparkFun-Coils:INDUCTOR-10UH
- LOGO1: value SPARKX-LOGO5 -> SFE_LOGO_NAME_FLAME.1_INCH; device 1.81_Greyscale_OLED_Breakout:SPARKX-LOGO5 -> SparkFun-Aesthetics:SFE_LOGO_NAME_FLAME.1_INCH
- U1: value AP3012 -> 1.25V 500mA; device 1.81_Greyscale_OLED_Breakout:AP3012 -> SparkFun-IC-Power:AP3012
Other:
- note added: "A. England"
- note added: "v01"
- note removed: "X11"
Changed lines of the file:
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@@
 <layers>
 <layer number="1" name="Top" color="4" fill="1" visible="no" active="no"/>
+<layer number="2" name="Route2" color="1" fill="3" visible="no" active="no"/>
+<layer number="3" name="Route3" color="4" fill="3" visible="no" active="no"/>
+<layer number="4" name="Route4" color="1" fill="4" visible="no" active="no"/>
+<layer number="5" name="Route5" color="4" fill="4" visible="no" active="no"/>
+<layer number="6" name="Route6" color="1" fill="8" visible="no" active="no"/>
+<layer number="7" name="Route7" color="4" fill="8" visible="no" active="no"/>
+<layer number="8" name="Route8" color="1" fill="2" visible="no" active="no"/>
+<layer number="9" name="Route9" color="4" fill="2" visible="no" active="no"/>
+<layer number="10" name="Route10" color="1" fill="7" visible="no" active="no"/>
+<layer number="11" name="Route11" color="4" fill="7" visible="no" active="no"/>
+<layer number="12" name="Route12" color="1" fill="5" visible="no" active="no"/>
+<layer number="13" name="Route13" color="4" fill="5" visible="no" active="no"/>
+<layer number="14" name="Route14" color="1" fill="6" visible="no" active="no"/>
+<layer number="15" name="Route15" color="4" fill="6" visible="no" active="no"/>
 <layer number="16" name="Bottom" color="1" fill="1" visible="no" active="no"/>
 <layer number="17" name="Pads" color="2" fill="1" visible="no" active="no"/>
@@
 <parts>
 <part name="FRAME1" library="SparkFun-Aesthetics" deviceset="FRAME-LETTER" device=""/>
-<part name="U1" library="1.81_Greyscale_OLED_Breakout" deviceset="AP3012" device=""/>
+<part name="U1" library="SparkFun-IC-Power" deviceset="AP3012" device="" value="1.25V 500mA"/>
 <part name="C1" library="SparkFun-Capacitors" deviceset="1.0UF" device="-0603-16V-10%" value="1.0uF"/>
-<part name="C2" library="SparkFun-Capacitors" deviceset="1.0UF" device="-0805-25V-(+80/-20%)" value="1.0uF/25V"/>
+<part name="C2" library="SparkFun-Capacitors" deviceset="1.0UF" device="-0805-25V-10%" value="1.0uF"/>
 <part name="R1" library="SparkFun-Resistors" deviceset="47KOHM" device="-0603-1/10W-1%" value="47k"/>
 <part name="R2" library="SparkFun-Resistors" deviceset="5.6KOHM" device="-0603-1/10W-1%" value="5.6k"/>
 <part name="D1" library="SparkFun-DiscreteSemi" deviceset="DIODE-SCHOTTKY" device="-BAT20J" value="1A/23V/620mV"/>
-<part name="L1" library="1.81_Greyscale_OLED_Breakout" deviceset="INDUCTOR" device="INDUCTOR_10UH" value="10uH"/>
+<part name="L1" library="SparkFun-Coils" deviceset="INDUCTOR" device="-10UH" value="10uH"/>
 <part name="SUPPLY1" library="SparkFun-PowerSymbols" deviceset="VIN" device=""/>
 <part name="GND1" library="SparkFun-PowerSymbols" deviceset="GND" device=""/>
@@
 <part name="SUPPLY14" library="SparkFun-PowerSymbols" deviceset="VIN" device=""/>
 <part name="J2" library="SparkFun-Connectors" deviceset="CONN_06" device="NO_SILK_NO_POP"/>
-<part name="LOGO1" library="1.81_Greyscale_OLED_Breakout" deviceset="SPARKX-LOGO" device="5" value="SPARKX-LOGO5"/>
+<part name="LOGO1" library="SparkFun-Aesthetics" deviceset="SFE_LOGO_NAME_FLAME" device=".1_INCH" value="SFE_LOGO_NAME_FLAME.1_INCH"/>
 <part name="H2" library="SparkFun-Hardware" deviceset="STAND-OFF" device=""/>
 <part name="FD1" library="SparkFun-Aesthetics" deviceset="FIDUCIAL" device="1X2"/>
 <part name="FD2" library="SparkFun-Aesthetics" deviceset="FIDUCIAL" device="1X2"/>
-<part name="DS1" library="1.81_Greyscale_OLED_Breakout" deviceset="OEL_1.8" device="OEL_Y3B" value="OEL_1.8OEL_Y3B"/>
+<part name="DS1" library="SparkFun-Displays" deviceset="OEL_1.8" device="OEL_Y3B" value="OEL_1.8OEL_Y3B"/>
+<part name="LOGO2" library="SparkFun-Aesthetics" deviceset="REVISION" device=""/>
+<part name="FD3" library="SparkFun-Aesthetics" deviceset="FIDUCIAL" device="1X2"/>
+<part name="FD4" library="SparkFun-Aesthetics" deviceset="FIDUCIAL" device="1X2"/>
+<part name="LOGO3" library="SparkFun-Aesthetics" deviceset="SFE_LOGO_FLAME" device=".1_INCH"/>
 </parts>
 <sheets>
@@
 <wire x1="73.66" y1="60.96" x2="147.32" y2="60.96" width="0.2032" layer="97" style="shortdash"/>
 <wire x1="73.66" y1="60.96" x2="73.66" y2="0" width="0.2032" layer="97" style="shortdash"/>
-<text x="238.76" y="7.62" size="2.54" layer="94">X11</text>
-<text x="172.72" y="10.16" size="2.54" layer="95">N. Seidle</text>
+<text x="238.76" y="7.62" size="2.54" layer="94">v01</text>
+<text x="170.18" y="11.176" size="2.54" layer="94">N. Seidle</text>
+<text x="174.498" y="7.112" size="2.54" layer="94">A. England</text>
 </plain>
 <instances>
@@
 <instance part="SUPPLY14" gate="G$1" x="200.66" y="111.76"/>
 <instance part="J2" gate="G$1" x="111.76" y="27.94" rot="MR0"/>
-<instance part="LOGO1" gate="G$1" x="38.1" y="27.94"/>
+<instance part="LOGO1" gate="G$1" x="7.62" y="17.78"/>
 <instance part="H2" gate="G$1" x="243.84" y="33.02"/>
 <instance part="FD1" gate="G$1" x="233.68" y="30.48"/>
 <instance part="FD2" gate="G$1" x="236.22" y="27.94"/>
 <instance part="DS1" gate="G$1" x="86.36" y="96.52"/>
+<instance part="LOGO2" gate="G$1" x="148.59" y="7.112"/>
+<instance part="FD3" gate="G$1" x="233.68" y="27.94"/>
+<instance part="FD4" gate="G$1" x="236.22" y="30.48"/>
+<instance part="LOGO3" gate="G$1" x="40.132" y="30.48"/>
 </instances>
 <busses>
