File: Hardware/1.81_Grayscale_OLED_Breakout.brd (EAGLE design)
At the start: 15.2 x 35.6 mm, 29 parts, among them U1 1.25V 500mA, U2 3.3V, U3 TXB0104

Commit message: post design review/checklist changes
Parts:
- added LOGO4: OSHW-LOGOS, SparkFun-Aesthetics:OSHW-LOGO-S
- added TP1: TEST-POINT2, SparkFun-Connectors:PAD.02X.02
Connections:
- net 12V: now also TP1.P$1
Routing:
- net 12V: track 20.8 -> 22.2 mm, vias 0 -> 1
- net N$2: track 5.72 -> 6.45 mm
- net VIN: track 53.5 -> 54.2 mm
Other:
- board text added: "1.81" Grayscale OLED Breakout"
- board text added: "Units in Inches"
- board text added: "VIN"
- board text removed: "1.81" Greyscale OLED Breakout"
- board text removed: "3.3-5V"
