File: Hardware/1.81_Grayscale_OLED_Breakout.sch (EAGLE design)
At the start: 29 parts, among them U1 1.25V 500mA, U2 3.3V, U3 TXB0104

Commit message: post design review/checklist changes
Parts:
- added LOGO4: OSHW-LOGOS, SparkFun-Aesthetics:OSHW-LOGOS
- added TP1: TEST-POINT2, SparkFun-Connectors:TEST-POINT2
- L1: device SparkFun-Coils:INDUCTOR-10UH -> SparkFun-Coils:INDUCTORINDUCTOR_10UH
Connections:
- net 12V: now also TP1.1
Changed lines of the file:
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@@
 <layer number="59" name="tCarbon" color="7" fill="1" visible="no" active="no"/>
 <layer number="60" name="bCarbon" color="7" fill="1" visible="no" active="no"/>
+<layer number="88" name="SimResults" color="9" fill="1" visible="yes" active="yes"/>
+<layer number="89" name="SimProbes" color="9" fill="1" visible="yes" active="yes"/>
 <layer number="90" name="Modules" color="5" fill="1" visible="yes" active="yes"/>
 <layer number="91" name="Nets" color="2" fill="1" visible="yes" active="yes"/>
@@
 <part name="R2" library="SparkFun-Resistors" deviceset="5.6KOHM" device="-0603-1/10W-1%" value="5.6k"/>
 <part name="D1" library="SparkFun-DiscreteSemi" deviceset="DIODE-SCHOTTKY" device="-BAT20J" value="1A/23V/620mV"/>
-<part name="L1" library="SparkFun-Coils" deviceset="INDUCTOR" device="-10UH" value="10uH"/>
+<part name="L1" library="SparkFun-Coils" deviceset="INDUCTOR" device="INDUCTOR_10UH" value="10uH"/>
 <part name="SUPPLY1" library="SparkFun-PowerSymbols" deviceset="VIN" device=""/>
 <part name="GND1" library="SparkFun-PowerSymbols" deviceset="GND" device=""/>
@@
 <part name="FD4" library="SparkFun-Aesthetics" deviceset="FIDUCIAL" device="1X2"/>
 <part name="LOGO3" library="SparkFun-Aesthetics" deviceset="SFE_LOGO_FLAME" device=".1_INCH"/>
+<part name="LOGO4" library="SparkFun-Aesthetics" deviceset="OSHW-LOGO" device="S"/>
+<part name="TP1" library="SparkFun-Connectors" deviceset="TEST-POINT" device="2"/>
 </parts>
 <sheets>
 <sheet>
 <plain>
-<text x="218.44" y="165.1" size="1.27" layer="97">VCC = 1.25 (1 + R1 / R2)
+<text x="218.44" y="165.1" size="1.27" layer="97" font="vector">VCC = 1.25 (1 + R1 / R2)
         = 1.25 (1+ 47/5.6)
         = 11.74 V</text>
-<text x="38.1" y="142.24" size="2.54" layer="97" align="top-center">VIN range: 2.6 - 5.5V
+<text x="38.1" y="142.24" size="2.54" layer="97" font="vector" align="top-center">VIN range: 2.6 - 5.5V
 (Low limit: AP3012,
 High limit: TXB0104)</text>
-<text x="2.54" y="180.34" size="2.54" layer="94">3.3V Voltage Regulator</text>
-<text x="149.86" y="180.34" size="2.54" layer="94">12V Boost</text>
-<text x="2.54" y="116.84" size="2.54" layer="94">1.81" Flexible OLED</text>
-<text x="149.86" y="119.38" size="2.54" layer="94">Level Shifting</text>
-<text x="76.2" y="55.88" size="2.54" layer="94">Pin Breakouts</text>
+<text x="2.54" y="180.34" size="2.54" layer="94" font="vector">3.3V Voltage Regulator</text>
+<text x="149.86" y="180.34" size="2.54" layer="94" font="vector">12V Boost</text>
+<text x="2.54" y="116.84" size="2.54" layer="94" font="vector">1.81" Flexible OLED</text>
+<text x="149.86" y="119.38" size="2.54" layer="94" font="vector">Level Shifting</text>
+<text x="76.2" y="55.88" size="2.54" layer="94" font="vector">Pin Breakouts</text>
 <wire x1="0" y1="124.46" x2="147.32" y2="124.46" width="0.2032" layer="97" style="shortdash"/>
 <wire x1="147.32" y1="124.46" x2="147.32" y2="185.42" width="0.2032" layer="97" style="shortdash"/>
@@
 <wire x1="73.66" y1="60.96" x2="147.32" y2="60.96" width="0.2032" layer="97" style="shortdash"/>
 <wire x1="73.66" y1="60.96" x2="73.66" y2="0" width="0.2032" layer="97" style="shortdash"/>
-<text x="238.76" y="7.62" size="2.54" layer="94">v01</text>
-<text x="170.18" y="11.176" size="2.54" layer="94">N. Seidle</text>
-<text x="174.498" y="7.112" size="2.54" layer="94">A. England</text>
+<text x="238.76" y="7.62" size="2.54" layer="94" font="vector">v01</text>
+<text x="172.72" y="11.176" size="2.54" layer="94" font="vector">N. Seidle</text>
+<text x="177.038" y="7.112" size="2.54" layer="94" font="vector">A. England</text>
 </plain>
 <instances>
@@
 <instance part="FD4" gate="G$1" x="236.22" y="30.48"/>
 <instance part="LOGO3" gate="G$1" x="40.132" y="30.48"/>
+<instance part="LOGO4" gate="G$1" x="35.56" y="12.7"/>
+<instance part="TP1" gate="G$1" x="220.98" y="160.02"/>
 </instances>
 <busses>
@@
 <pinref part="C2" gate="G$1" pin="1"/>
 <wire x1="205.74" y1="167.64" x2="215.9" y2="167.64" width="0.1524" layer="91"/>
-<wire x1="215.9" y1="167.64" x2="215.9" y2="154.94" width="0.1524" layer="91"/>
+<wire x1="215.9" y1="167.64" x2="215.9" y2="160.02" width="0.1524" layer="91"/>
 <pinref part="SUPPLY2" gate="G$1" pin="12V"/>
+<wire x1="215.9" y1="160.02" x2="215.9" y2="154.94" width="0.1524" layer="91"/>
 <wire x1="215.9" y1="167.64" x2="215.9" y2="170.18" width="0.1524" layer="91"/>
 <junction x="215.9" y="167.64"/>
-</segment>
-<segment>
+<pinref part="TP1" gate="G$1" pin="1"/>
+<wire x1="220.98" y1="160.02" x2="215.9" y2="160.02" width="0.1524" layer="91"/>
+<junction x="215.9" y="160.02"/>
+</segment>
+<segment>
