File: Hardware/1.81_Grayscale_OLED_Breakout.sch (EAGLE design)
At the start: 31 parts, among them U1 1.25V 500mA, U2 3.3V, U3 TXB0104

Commit message: added panel
Parts:
- removed TP1: TEST-POINT2, SparkFun-Connectors:TEST-POINT2
- L1: device SparkFun-Coils:INDUCTORINDUCTOR_10UH -> SparkFun-Coils:INDUCTOR-CDRH-10UH
Connections:
- net 12V: no longer TP1.1
Changed lines of the file:
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@@
 <part name="R2" library="SparkFun-Resistors" deviceset="5.6KOHM" device="-0603-1/10W-1%" value="5.6k"/>
 <part name="D1" library="SparkFun-DiscreteSemi" deviceset="DIODE-SCHOTTKY" device="-BAT20J" value="1A/23V/620mV"/>
-<part name="L1" library="SparkFun-Coils" deviceset="INDUCTOR" device="INDUCTOR_10UH" value="10uH"/>
+<part name="L1" library="SparkFun-Coils" deviceset="INDUCTOR" device="-CDRH-10UH" value="10uH"/>
 <part name="SUPPLY1" library="SparkFun-PowerSymbols" deviceset="VIN" device=""/>
 <part name="GND1" library="SparkFun-PowerSymbols" deviceset="GND" device=""/>
@@
 <part name="LOGO3" library="SparkFun-Aesthetics" deviceset="SFE_LOGO_FLAME" device=".1_INCH"/>
 <part name="LOGO4" library="SparkFun-Aesthetics" deviceset="OSHW-LOGO" device="S"/>
-<part name="TP1" library="SparkFun-Connectors" deviceset="TEST-POINT" device="2"/>
 </parts>
 <sheets>
@@
 <instance part="LOGO3" gate="G$1" x="40.132" y="30.48"/>
 <instance part="LOGO4" gate="G$1" x="35.56" y="12.7"/>
-<instance part="TP1" gate="G$1" x="220.98" y="160.02"/>
 </instances>
 <busses>
@@
 <pinref part="C2" gate="G$1" pin="1"/>
 <wire x1="205.74" y1="167.64" x2="215.9" y2="167.64" width="0.1524" layer="91"/>
-<wire x1="215.9" y1="167.64" x2="215.9" y2="160.02" width="0.1524" layer="91"/>
+<wire x1="215.9" y1="167.64" x2="215.9" y2="154.94" width="0.1524" layer="91"/>
 <pinref part="SUPPLY2" gate="G$1" pin="12V"/>
-<wire x1="215.9" y1="160.02" x2="215.9" y2="154.94" width="0.1524" layer="91"/>
 <wire x1="215.9" y1="167.64" x2="215.9" y2="170.18" width="0.1524" layer="91"/>
 <junction x="215.9" y="167.64"/>
-<pinref part="TP1" gate="G$1" pin="1"/>
-<wire x1="220.98" y1="160.02" x2="215.9" y2="160.02" width="0.1524" layer="91"/>
-<junction x="215.9" y="160.02"/>
-</segment>
-<segment>
+</segment>
+<segment>

Commit message: post checklist changes
Parts:
- added TP1, TP2, TP3, TP4, TP5, TP6, TP7: TEST-POINT3, SparkFun-Connectors:TEST-POINT3
- U1: value 1.25V 500mA -> AP3012
Connections:
- net !CS!: now also TP2.1
- net !RES!: now also TP1.1
- net 12V: now also TP7.1
- net 3.3V: now also TP6.1
- net N$1: now also TP5.1
- net SCLK: now also TP3.1
- net SDIN: now also TP4.1
Other:
- note added: "v10"
- note removed: "v01"
- moved on the sheet: C3, C4, C5, C6
